File: POE-PD-NETWORK.kicad_pcb (KiCad board)
At the start: 6 copper layers, 11 parts, among them J1 8P8C-NE8FBH-C5-S

Commit message: Update kicad schematic to use three blocks to make the schematic more understandable and lock in pcb board requirements.
Other:
- copper layers 6 -> 8
Changed lines of the file:
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@@
 	(generator_version "10.0")
 	(general
-		(thickness 1.6)
+		(thickness 2.456)
 		(legacy_teardrops no)
 	)
@@
 	(layers
 		(0 "F.Cu" signal)
-		(4 "In1.Cu" signal)
-		(6 "In2.Cu" signal)
-		(8 "In3.Cu" signal)
-		(10 "In4.Cu" signal)
-		(2 "B.Cu" signal)
+		(4 "In1.Cu" power)
+		(6 "In2.Cu" power)
+		(8 "In3.Cu" power)
+		(10 "In4.Cu" power)
+		(12 "In5.Cu" power)
+		(14 "In6.Cu" signal)
+		(2 "B.Cu" power)
 		(9 "F.Adhes" user "F.Adhesive")
 		(11 "B.Adhes" user "B.Adhesive")
@@
 			(layer "F.Mask"
 				(type "Top Solder Mask")
-				(thickness 0.01)
+				(thickness 0.025)
+				(material "LPI Green, IPC-SM-840E Class H, >46kv/mm, Meet or exceed spec")
+				(epsilon_r 3.8)
+				(loss_tangent 0.025)
 			)
 			(layer "F.Cu"
@@
 			(layer "dielectric 1"
 				(type "prepreg")
-				(thickness 0.1)
-				(material "FR4")
-				(epsilon_r 4.5)
-				(loss_tangent 0.02)
+				(thickness 0.254)
+				(material "Isola 550H")
+				(epsilon_r 4.43)
+				(loss_tangent 0.014)
 			)
 			(layer "In1.Cu"
 				(type "copper")
-				(thickness 0.035)
+				(thickness 0.07)
 			)
 			(layer "dielectric 2"
-				(type "prepreg")
-				(thickness 0.535)
-				(material "FR4")
-				(epsilon_r 4.5)
-				(loss_tangent 0.02)
+				(type "core")
+				(thickness 0.3)
+				(material "Isola 550H")
+				(epsilon_r 4.43)
+				(loss_tangent 0.014)
 			)
 			(layer "In2.Cu"
 				(type "copper")
-				(thickness 0.035)
+				(thickness 0.07)
 			)
 			(layer "dielectric 3"
 				(type "prepreg")
-				(thickness 0.1)
-				(material "FR4")
-				(epsilon_r 4.5)
-				(loss_tangent 0.02)
+				(thickness 0.254)
+				(material "Isola 550H")
+				(epsilon_r 4.43)
+				(loss_tangent 0.014)
 			)
 			(layer "In3.Cu"
 				(type "copper")
-				(thickness 0.035)
+				(thickness 0.07)
 			)
 			(layer "dielectric 4"
 				(type "core")
-				(thickness 0.535)
-				(material "FR4")
-				(epsilon_r 4.5)
-				(loss_tangent 0.02)
+				(thickness 0.3)
+				(material "Isola 550H")
+				(epsilon_r 4.43)
+				(loss_tangent 0.014)
 			)
 			(layer "In4.Cu"
 				(type "copper")
-				(thickness 0.035)
+				(thickness 0.07)
 			)
 			(layer "dielectric 5"
 				(type "prepreg")
-				(thickness 0.1)
-				(material "FR4")
-				(epsilon_r 4.5)
-				(loss_tangent 0.02)
+				(thickness 0.254)
+				(material "Isola 550H")
+				(epsilon_r 4.43)
+				(loss_tangent 0.014)
+			)
+			(layer "In5.Cu"
+				(type "copper")
+				(thickness 0.07)
+			)
+			(layer "dielectric 6"
+				(type "core")
+				(thickness 0.3)
+				(material "Isola 550H")
+				(epsilon_r 4.43)
+				(loss_tangent 0.014)
+			)
+			(layer "In6.Cu"
+				(type "copper")
+				(thickness 0.035)
+			)
+			(layer "dielectric 7"
+				(type "prepreg")
+				(thickness 0.254)
+				(material "Isola 550H")
+				(epsilon_r 4.43)
+				(loss_tangent 0.014)
 			)
 			(layer "B.Cu"
 				(type "copper")
-				(thickness 0.035)
+				(thickness 0.07)
 			)
 			(layer "B.Mask"
 				(type "Bottom Solder Mask")
-				(thickness 0.01)
+				(thickness 0.025)
+				(material "LPI Green, IPC-SM-840E Class H, >46kv/mm, Meet or exceed spec")
+				(epsilon_r 3.8)
+				(loss_tangent 0.025)
 			)
 			(layer "B.Paste"
@@
 		(capping no)
 		(filling no)
+		(zone_defaults)
 		(pcbplotparams
 			(layerselection 0x00000000_00000000_55555555_5755f5ff)
