File: clean_side_(pre_voltage_mux,_supercaps._incl._mux).kicad_sch (KiCad schematic)
At the start: 0 parts

Commit message: Update kicad schematic to use three blocks to make the schematic more understandable and lock in pcb board requirements.
Other:
- title: POE-PD-NETWORK Schematic - Dirty Side, Isolated -> POE-PD-NETWORK Schematic - Clean Side Pre voltage mux
Changed lines of the file:
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@@
 	(paper "A4")
 	(title_block
-		(title "POE-PD-NETWORK Schematic - Dirty Side, Isolated")
+		(title "POE-PD-NETWORK Schematic - Clean Side Pre voltage mux")
 		(rev "V0.1-WIP")
 		(company "Copyright © 2026 Coconut Nivrinu Squirt")
@@
 	(sheet_instances
 		(path "/"
-			(page "1")
+			(page "2")
 		)
 	)
